File: schematics/fc/fc.sch (KiCad schematic (older format))
At the start: 47 parts

Commit message: Restructure schematics; finish FC/Radio
Parts:
- removed C?: 100n, agg:0402, symbol cusf-kicad:C
- removed C?: 100n, symbol cusf-kicad:C
- removed D?: D, agg:SOD-323, symbol cusf-kicad:D
- removed D?: GRN, agg:0603-LED, symbol cusf-kicad:LED
- removed D?: RED, agg:0603-LED, symbol cusf-kicad:LED
- removed J?: TC1, symbol cusf-kicad:CONN_01x02
- removed J?: TC4, symbol cusf-kicad:CONN_01x02
- removed J?: TC3, symbol cusf-kicad:CONN_01x02
- removed J?: TC2, symbol cusf-kicad:CONN_01x02
- removed J?: PT2, symbol cusf-kicad:CONN_01x02
- removed J?: PT1, symbol cusf-kicad:CONN_01x02
- removed J?: CAMERA, symbol cusf-kicad:CONN_02x12
- removed LS?: SOUNDER, agg:KSSG13J12-N, symbol cusf-kicad:SOUNDER
- removed P?: SWD_TC, agg:TC2030-NL, symbol cusf-kicad:SWD_TC
- removed Q?: NFET, agg:SOT-23, symbol cusf-kicad:NFET
- removed R? (x3): 100, agg:0402, symbol cusf-kicad:R
- added C? (x5): 100n, symbol cusf-kicad:C
- added C? (x6): 1u, symbol cusf-kicad:C
- added C?: 200n, symbol cusf-kicad:C
- added C?: 100p, symbol cusf-kicad:C
- added C?: 2.2u, symbol cusf-kicad:C
- added C?: 220p, symbol cusf-kicad:C
- added C?: 200p, symbol cusf-kicad:C
- added C? (x2): 2µ2, agg:0402, symbol cusf-kicad:C
- added C? (x6): 100n, agg:0402, symbol cusf-kicad:C
- added C?: 1µ, agg:0402, symbol cusf-kicad:C
- added C?: 4µ7, agg:0402, symbol cusf-kicad:C
- added C?: 1p2, symbol cusf-kicad:C
- added C? (x2): 3p, symbol cusf-kicad:C
- added C? (x4): 3p3, symbol cusf-kicad:C
- added C?: 5p1, symbol cusf-kicad:C
- added C?: 6n8, symbol cusf-kicad:C
- added C?: 1p, symbol cusf-kicad:C
- added C?: 4p7, symbol cusf-kicad:C
- added C?: 6n2, symbol cusf-kicad:C
- added D? (x2): GRN, agg:0603-LED, symbol cusf-kicad:LED
- added D? (x2): RED, agg:0603-LED, symbol cusf-kicad:LED
- added D?: YLW, agg:0603-LED, symbol cusf-kicad:LED
- added IC?: SN74LVC1G0832, agg:SC-70-6, symbol cusf-kicad:SN74LVC1G0832
- added IC?: Si4463, agg:QFN-20-EP-SI, symbol cusf-kicad:Si4460
- added IC?: NCP4620, agg:SC-70-5, symbol cusf-kicad:NCP4620
- added IC?: BGM1043N7, agg:DFN-6-EP-BGM, symbol cusf-kicad:BGM1043N7
- added IC?: NCP380, agg:DFN-6-EP-ONSEMI, symbol cusf-kicad:NCP380
- added IC?: MAX-M8Q, agg:MAX-M8Q, symbol cusf-kicad:MAX-M8Q
- added IC?: STM32F405RxTx, agg:LQFP-64, symbol cusf-kicad:STM32F405RxTx
- added IC?: MCP2562, agg:DFN-8-EP-MICROCHIP, symbol cusf-kicad:MCP2562
- added IC?: SL18860DC, cusf:DFN-10-SL18860DC, symbol cusf-kicad:SL18860DC
- added L?: 9n1, symbol cusf-kicad:L
- added L?: 8n2, symbol cusf-kicad:L
- added L? (x3): 92n, symbol cusf-kicad:L
- added L? (x3): 91n, symbol cusf-kicad:L
- added L?: 120n, symbol cusf-kicad:L
- added L? (x2): 24n, symbol cusf-kicad:L
- added L? (x2): 18n, symbol cusf-kicad:L
- added L? (x2): 3n3, symbol cusf-kicad:L
- added L? (x2): 12n, symbol cusf-kicad:L
- added L?: 100n, symbol cusf-kicad:L
- added L? (x2): 22n, symbol cusf-kicad:L
- added L? (x2): 11n, symbol cusf-kicad:L
- added R? (x5): 100, agg:0402, symbol cusf-kicad:R
- added R? (x2): 10k, symbol cusf-kicad:R
- added R?: 110k, symbol cusf-kicad:R
- added R?: 10, symbol cusf-kicad:R
- added Y?: TCXO, symbol cusf-kicad:TCXO
Connections:
- net labels added: 1v8, ACCEL_MISO, ACCEL_MOSI, ANT_~EN, ANT_~FLAG, BARO_MISO, BARO_MOSI, FC_LED_GRN, FC_LED_RED, FC_LED_YLW, FC_MCU_CLK, GPS, GPS_PPS, GPS_RESET_N, GPS_RX, GPS_TP, GPS_TX, MCU_CLK, RADIO_CLK, RADIO_GATE, RADIO_GPIO1, RADIO_LED_GRN, RADIO_LED_RED, RADIO_LED_YLW, RADIO_MCU_CLK, RADIO_SCLK, RADIO_SDI, RADIO_SDN, RADIO_SDO, RADIO_nIRQ, RADIO_nSEL, RXn, RXp, TX
- net labels removed: ACCEL_SDI, ACCEL_SDO, BARO_DIN, BARO_DOUT, BEEPER, DCMI_D0, DCMI_D1, DCMI_D2, DCMI_D3, DCMI_D4, DCMI_D5, DCMI_D6, DCMI_D7, DCMI_HSYNC, DCMI_NRST, DCMI_PIXCLK, DCMI_PWR_EN, DCMI_SCL, DCMI_SDA, DCMI_VSYNC, LED_GRN, LED_RED, LED_YLW, P1+, P1-, P2+, P2-, T1+, T1-, T2+, T2-, T3+, T3-, T4+, T4-, VCC
- wire segments 237 -> 490
- no-connect marks 34 -> 69
Other:
- note added: "Accelerometer"
- note added: "Antennas"
- note added: "Barometer"
- note added: "Clock Distribution"
- note added: "FLIGHT COMPUTER"
- note added: "GPS"
- note added: "Lowpass Filter"
- note added: "Microcontroller"
- note added: "PA Match/Filter (868 MHz)"
- note added: "PA Match/Filter (915 MHz)"
- note added: "PB4 is JTRST,\nDO NOT CONNECT\n(Errata 2.1.4)"
- note added: "RADIO"
- note added: "TODO:\n- Check all label names, correctly label duplicated ones\n (e.g. CAN, JTAG)"
- note added: "Telemetry Radio"
- note added: "What's going on here?\n\nWe have two subsystems we could slot in here, depending on the design frequency.\n\nTo the right you'll find match/filter circuits for both 868 and 915 MHz.\nChoose wisely."
- note added: "https://www.silabs.com/documents/public/application-notes/AN648.pdf"
- note removed: "ACCELEROMETER"
- note removed: "BAROMETER"
- note removed: "BEEPER"
- note removed: "MICROCONTROLLER"
- note removed: "NOTE: BEEPER moved\nfrom PA0 to PA3\n- can we do this?"
- note removed: "PB4 is JTRST, DO NOT CONNECT (Errata 2.1.4)"
- moved on the sheet: C?, D?, IC?, P?, R?, Y?

Commit message: Move dl to blackbox; fix minor errors in fc
Parts:
- removed C? (x2): 10p, agg:0402, symbol cusf-kicad:C
- removed R?: 100, agg:0402, symbol cusf-kicad:R
- removed Y?: 26M, agg:XTAL-20x16, symbol cusf-kicad:SMD_XTAL
Connections:
- net MCU_CLK is gone; now on net RADIO_MCU_CLK: IC?.5 (PH0)
- net FC_MCU_CLK: now also IC?.5 (PH0)
- net GND: no longer C?.1, C?.1, C?.1, C?.1, C?.1, C?.1, C?.1, C?.1, C?.1, IC?.12 (VSSA), IC?.18 (VSS), IC?.60 (BOOT0), IC?.63 (VSS)
- new net: C?.1, C?.1, C?.1, C?.1, C?.1, C?.1, C?.1, C?.1, C?.1, IC?.12 (VSSA), IC?.18 (VSS), IC?.60 (BOOT0), IC?.63 (VSS)
- no-connect marks 69 -> 70
Other:
- moved on the sheet: C?, D?, IC?, P?
