File: schematics/flight-computer/transceivers.sch (KiCad schematic (older format))
At the start: 4 parts

Commit message: Add temp rescue symbol while switching libs
Parts:
- IC?: symbol cusf-kicad:SN65LVDT41 -> flight-computer-rescue:SN65LVDT41-cusf-kicad
Changed lines of the file:
@@
 	6700 4100 8500 4100
 $Comp
-L cusf-kicad:SN65LVDT41 IC?
+L flight-computer-rescue:SN65LVDT41-cusf-kicad IC?
 U 1 1 62044C5D
 P 4650 3150
