File: schematics/02 flight-computer/flight-computer.kicad_sch (KiCad schematic)
At the start: 46 parts, among them J1 SWD, J2 PWR, J3 GND CTRL, J4 RADIO, J5 PYRO, J6 DATALOGGER, J7 BLACKBOX, U1 MAX14787E, U2 STM32F405RGT6, U3 MAX14787E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

Commit message: Minor schematic revisions
Parts:
- D1, D2: footprint Strix:LED_0402 -> Strix:LED_0603
- J2: footprint (none) -> Strix:Molex_Nano-Fit_105313-1104
- J4, J5, J6: footprint (none) -> Strix:Molex_Nano-Fit_105314-1110
Connections:
- net IMU_SDN: now also U2.27 (PB1)
- net I2C1_SCL: no longer names the net of U2.58 (PB6)
- net I2C1_SDA: no longer names the net of U2.59 (PB7)
- net SPI3_MISO: no longer names the net of U2.52 (PC11)
- net SPI3_MOSI: no longer names the net of U2.53 (PC12)
- net SPI3_SCLK: no longer names the net of U2.51 (PC10)
- no-connect marks 21 -> 25
Changed lines of the file:
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@@
     (title "PROJECT STRIX: MCU board")
     (date "2022-09-03")
-    (rev "1.3.2")
+    (rev "1.3.3")
     (company "Cambridge University Spaceflight")
     (comment 1 "Drawn by H. Franks")
@@
   (junction (at 88.9 49.53) (diameter 0) (color 0 0 0 0)
   )
-  (no_connect (at 115.57 95.25))
   (no_connect (at 115.57 107.95))
   (no_connect (at 115.57 130.81))
@@
   (no_connect (at 115.57 49.53))
   (no_connect (at 115.57 90.17))
+  (no_connect (at 115.57 118.11))
+  (no_connect (at 115.57 115.57))
+  (no_connect (at 115.57 113.03))
   (no_connect (at 90.17 133.35))
   (no_connect (at 115.57 67.31))
@@
   (no_connect (at 115.57 123.19))
   (no_connect (at 115.57 125.73))
-  (no_connect (at 115.57 46.99))
+  (no_connect (at 115.57 95.25))
   (no_connect (at 115.57 92.71))
   (no_connect (at 90.17 120.65))
   (no_connect (at 46.99 127))
+  (no_connect (at 115.57 62.23))
+  (no_connect (at 115.57 59.69))
   (no_connect (at 115.57 64.77))
   (no_connect (at 90.17 118.11))
@@
     (stroke (width 0) (type default) (color 0 0 0 0))
   )
-  (polyline (pts (xy 48.26 54.61) (xy 88.9 54.61))
+  (polyline (pts (xy 58.42 54.61) (xy 88.9 54.61))
     (stroke (width 0.1) (type dot) (color 0 194 0 1))
   )
@@
     (stroke (width 0) (type default) (color 0 0 0 0))
   )
-  (polyline (pts (xy 48.26 52.07) (xy 88.9 52.07))
+  (polyline (pts (xy 58.42 52.07) (xy 88.9 52.07))
     (stroke (width 0.1) (type dot) (color 0 194 0 1))
   )
@@
     (stroke (width 0) (type dot) (color 0 0 0 0))
   )
+  (wire (pts (xy 115.57 46.99) (xy 132.08 46.99))
+    (stroke (width 0) (type default) (color 0 0 0 0))
+  )
   (polyline (pts (xy 21.59 29.21) (xy 21.59 142.24))
     (stroke (width 0) (type default) (color 0 0 0 0))
@@
     (stroke (width 0) (type default) (color 0 0 0 0))
   )
-  (polyline (pts (xy 48.26 46.99) (xy 88.9 46.99))
+  (polyline (pts (xy 58.42 46.99) (xy 88.9 46.99))
     (stroke (width 0.1) (type dot) (color 0 194 0 1))
   )
@@
     (stroke (width 0) (type dot) (color 0 0 0 0))
   )
-  (polyline (pts (xy 48.26 49.53) (xy 88.9 49.53))
+  (polyline (pts (xy 58.42 49.53) (xy 88.9 49.53))
     (stroke (width 0.1) (type dot) (color 0 194 0 1))
   )
@@
     (stroke (width 0) (type default) (color 0 0 0 0))
   )
-  (wire (pts (xy 115.57 62.23) (xy 132.08 62.23))
-    (stroke (width 0) (type default) (color 0 0 0 0))
-  )
   (wire (pts (xy 214.63 123.19) (xy 215.9 123.19))
     (stroke (width 0) (type default) (color 0 0 0 0))
@@
     (stroke (width 0) (type default) (color 0 0 0 0))
   )
-  (wire (pts (xy 115.57 113.03) (xy 132.08 113.03))
-    (stroke (width 0) (type default) (color 0 0 0 0))
-  )
   (polyline (pts (xy 231.14 68.58) (xy 231.14 95.25))
     (stroke (width 0) (type dot) (color 0 0 0 0))
   )
-  (wire (pts (xy 115.57 115.57) (xy 132.08 115.57))
-    (stroke (width 0) (type default) (color 0 0 0 0))
-  )
   (wire (pts (xy 77.47 57.15) (xy 88.9 57.15))
     (stroke (width 0) (type default) (color 0 0 0 0))
@@
     (stroke (width 0) (type default) (color 0 0 0 0))
   )
-  (wire (pts (xy 115.57 59.69) (xy 132.08 59.69))
-    (stroke (width 0) (type default) (color 0 0 0 0))
-  )
   (wire (pts (xy 96.52 161.29) (xy 99.06 161.29))
     (stroke (width 0) (type default) (color 0 0 0 0))
@@
     (stroke (width 0) (type default) (color 0 0 0 0))
   )
-  (polyline (pts (xy 48.26 44.45) (xy 88.9 44.45))
+  (polyline (pts (xy 58.42 44.45) (xy 88.9 44.45))
     (stroke (width 0.1) (type dot) (color 0 194 0 1))
   )
@@
     (stroke (width 0) (type default) (color 0 0 0 0))
   )
-  (wire (pts (xy 115.57 118.11) (xy 132.08 118.11))
-    (stroke (width 0) (type default) (color 0 0 0 0))
-  )
   (polyline (pts (xy 139.7 29.21) (xy 139.7 142.24))
     (stroke (width 0) (type default) (color 0 0 0 0))
@@
     (effects (font (size 1.27 1.27)) (justify right bottom))
   )
-  (label "I2C1_SCL" (at 132.08 59.69 180)
+  (label "IMU_SDN" (at 132.08 46.99 180)
     (effects (font (size 1.27 1.27)) (justify right bottom))
   )
@@
     (effects (font (size 1.27 1.27)) (justify right bottom))
   )
-  (label "I2C1_SDA" (at 132.08 62.23 180)
-    (effects (font (size 1.27 1.27)) (justify right bottom))
-  )
   (label "RADIO_SDN" (at 132.08 105.41 180)
     (effects (font (size 1.27 1.27)) (justify right bottom))
@@
     (effects (font (size 1.27 1.27)) (justify left bottom))
   )
-  (label "SPI3_MISO" (at 132.08 115.57 180)
-    (effects (font (size 1.27 1.27)) (justify right bottom))
-  )
   (label "IMU_INT" (at 270.51 80.01 180)
     (effects (font (size 1.27 1.27)) (justify right bottom))
@@
     (effects (font (size 1.27 1.27)) (justify right bottom))
   )
-  (label "SPI3_MOSI" (at 132.08 118.11 180)
-    (effects (font (size 1.27 1.27)) (justify right bottom))
-  )
   (label "SWDCLK" (at 74.93 130.81 0)
     (effects (font (size 1.27 1.27)) (justify left bottom))
@@
     (effects (font (size 1.27 1.27)) (justify left bottom))
   )
-  (label "SPI3_SCLK" (at 132.08 113.03 180)
-    (effects (font (size 1.27 1.27)) (justify right bottom))
-  )
   (label "NRST" (at 55.88 129.54 180)
     (effects (font (size 1.27 1.27)) (justify right bottom))
@@
       (effects (font (size 1.27 1.27)) (justify left))
     )
-    (property "Footprint" "" (id 2) (at 198.12 52.07 0)
+    (property "Footprint" "Strix:Molex_Nano-Fit_105313-1104" (id 2) (at 198.12 52.07 0)
       (effects (font (size 1.27 1.27)) hide)
     )
@@
       (effects (font (size 1.27 1.27)) (justify left))
     )
-    (property "Footprint" "Strix:LED_0402" (id 2) (at 163.83 130.81 0)
+    (property "Footprint" "Strix:LED_0603" (id 2) (at 163.83 130.81 0)
       (effects (font (size 1.27 1.27)) hide)
     )
@@
     (property "Reference" "J5" (id 0) (at 251.46 43.18 0))
     (property "Value" "PYRO" (id 1) (at 251.46 45.72 0))
-    (property "Footprint" "" (id 2) (at 250.19 54.61 0)
+    (property "Footprint" "Strix:Molex_Nano-Fit_105314-1110" (id 2) (at 250.19 54.61 0)
       (effects (font (size 1.27 1.27)) hide)
     )
@@
       (effects (font (size 1.27 1.27)) (justify left))
     )
-    (property "Footprint" "Strix:LED_0402" (id 2) (at 151.13 130.81 0)
+    (property "Footprint" "Strix:LED_0603" (id 2) (at 151.13 130.81 0)
       (effects (font (size 1.27 1.27)) hide)
     )
@@
     (property "Reference" "J6" (id 0) (at 251.46 71.12 0))
     (property "Value" "DATALOGGER" (id 1) (at 251.46 73.66 0))
-    (property "Footprint" "" (id 2) (at 250.19 82.55 0)
+    (property "Footprint" "Strix:Molex_Nano-Fit_105314-1110" (id 2) (at 250.19 82.55 0)
       (effects (font (size 1.27 1.27)) hide)
     )
@@
     (property "Reference" "J4" (id 0) (at 209.55 71.12 0))
     (property "Value" "RADIO" (id 1) (at 209.55 73.66 0))
-    (property "Footprint" "" (id 2) (at 208.28 82.55 0)
+    (property "Footprint" "Strix:Molex_Nano-Fit_105314-1110" (id 2) (at 208.28 82.55 0)
       (effects (font (size 1.27 1.27)) hide)
     )
@@
     )
     (path "/4f1e5aa6-2eb5-4a86-8556-a7c4a7bcd0d6"
-      (reference "D1") (unit 1) (value "YLW") (footprint "Strix:LED_0402")
+      (reference "D1") (unit 1) (value "YLW") (footprint "Strix:LED_0603")
     )
     (path "/2d083f8a-638e-4090-9ef1-dff744bfe3b2"
-      (reference "D2") (unit 1) (value "RED") (footprint "Strix:LED_0402")
+      (reference "D2") (unit 1) (value "RED") (footprint "Strix:LED_0603")
     )
     (path "/be6fff45-19e4-4b71-a23e-5ad221ed2b84"
@@
     )
     (path "/241a6b77-76c6-4d56-a39b-77de140470e8"
-      (reference "J2") (unit 1) (value "PWR") (footprint "")
+      (reference "J2") (unit 1) (value "PWR") (footprint "Strix:Molex_Nano-Fit_105313-1104")
     )
     (path "/b4f653be-4121-4a5f-9d0b-f42e3b0395a1"
@@
     )
     (path "/c6520e67-b2c8-4991-962a-524aa423f8d3"
-      (reference "J4") (unit 1) (value "RADIO") (footprint "")
+      (reference "J4") (unit 1) (value "RADIO") (footprint "Strix:Molex_Nano-Fit_105314-1110")
     )
     (path "/4d9cb1c8-c634-4a61-bb1f-c4a2eaf2ff92"
-      (reference "J5") (unit 1) (value "PYRO") (footprint "")
+      (reference "J5") (unit 1) (value "PYRO") (footprint "Strix:Molex_Nano-Fit_105314-1110")
     )
     (path "/7116de53-c7c3-4aaa-a474-e6e3379b3761"
-      (reference "J6") (unit 1) (value "DATALOGGER") (footprint "")
+      (reference "J6") (unit 1) (value "DATALOGGER") (footprint "Strix:Molex_Nano-Fit_105314-1110")
     )
     (path "/d918eba2-1f12-4557-b5ed-a1c2fae655d3"

Commit message: Further schematic work
Parts:
- removed J5: PYRO, Strix:Molex_Nano-Fit_105314-1110, symbol Strix:Conn_02x05
- added J?: PYRO, symbol Strix:Conn_02x03
Connections:
- net GND: now also J?.6 (Pin_6)
- net PYRO1_EN: now also J?.2 (Pin_2)
- net PYRO2_EN: now also J?.4 (Pin_4)
- net PYRO3_EN: now also J?.1 (Pin_1)
- net PYRO4_EN: now also J?.3 (Pin_3)
- new net ARM: J?.5 (Pin_5)
Other:
- moved on the sheet: C1, C10, C11, C12, C13, C14, C15, C2, C3, C4, C5, C6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
